Commit message: Replace custom 5-DOF arm with official KBot 20-DOF humanoid model
- Add official URDF from kscalelabs/kbot-models with package:// mesh paths
- Add 24 STL meshes from kscalelabs/kbot-models
- Rewrite steveros.urdf.xacro as thin wrapper: includes kbot.urdf + ros2_control
- Rewrite ros2_control xacro with all 20 joints (motor_id, sign, limits)
- Split controllers into 4 per-limb JointTrajectoryControllers (TALOS pattern)
- Update launch file to spawn right_arm, left_arm, right_leg, left_leg controllers
- Update descriptions and comments for 20-DOF humanoid

Co-Authored-By: Claude Opus 4.6 <noreply@anthropic.com>

File: steveros_description/urdf/steveros.urdf.xacro (robot description, xacro)
@@ -1,108 +1,8 @@
 <?xml version="1.0"?>
 <robot xmlns:xacro="http://www.ros.org/wiki/xacro" name="steveros">
-  <!-- Cylinder geometry for all links (replace with K-Scale STL meshes later) -->
-  <xacro:macro name="arm_link" params="name length:=0.1 radius:=0.025">
-    <link name="${name}">
-      <visual>
-        <geometry>
-          <cylinder length="${length}" radius="${radius}"/>
-        </geometry>
-        <origin xyz="0 0 ${-length/2}" rpy="0 0 0"/>
-        <material name="grey">
-          <color rgba="0.5 0.5 0.5 1.0"/>
-        </material>
-      </visual>
-      <collision>
-        <geometry>
-          <cylinder length="${length}" radius="${radius}"/>
-        </geometry>
-        <origin xyz="0 0 ${-length/2}" rpy="0 0 0"/>
-      </collision>
-      <inertial>
-        <mass value="0.5"/>
-        <inertia ixx="0.001" ixy="0" ixz="0" iyy="0.001" iyz="0" izz="0.001"/>
-      </inertial>
-    </link>
-  </xacro:macro>
-  <!-- Base link (fixed) -->
-  <link name="base_link">
-    <visual>
-      <geometry>
-        <cylinder length="0.05" radius="0.04"/>
-      </geometry>
-      <material name="dark_grey">
-        <color rgba="0.3 0.3 0.3 1.0"/>
-      </material>
-    </visual>
-    <collision>
-      <geometry>
-        <cylinder length="0.05" radius="0.04"/>
-      </geometry>
-    </collision>
-    <inertial>
-      <mass value="1.0"/>
-      <inertia ixx="0.01" ixy="0" ixz="0" iyy="0.01" iyz="0" izz="0.01"/>
-    </inertial>
-  </link>
-  <!-- Arm links -->
-  <xacro:arm_link name="shoulder_pitch_link" length="0.08" radius="0.03"/>
-  <xacro:arm_link name="shoulder_roll_link" length="0.14" radius="0.025"/>
-  <xacro:arm_link name="elbow_link" length="0.14" radius="0.022"/>
-  <xacro:arm_link name="wrist_pitch_link" length="0.10" radius="0.018"/>
-  <xacro:arm_link name="wrist_roll_link" length="0.06" radius="0.015"/>
-  <!-- End-effector (virtual) -->
-  <link name="end_effector_link"/>
-  <!--
-    Joint chain from kbot URDF (kscalelabs/kbot-models kbot/robot.urdf)
-    Origins and axes match kinematics.py:_JOINT_CHAIN exactly.
-    Limits from config.yaml converted to radians.
-  -->
-  <!-- Joint 1: shoulder_pitch (URDF: dof_right_shoulder_pitch_03) -->
-  <joint name="shoulder_pitch_joint" type="revolute">
-    <parent link="base_link"/>
-    <child link="shoulder_pitch_link"/>
-    <origin xyz="-0.120999 0.002025 0.336659" rpy="0 ${-pi/2} 0"/>
-    <axis xyz="0 0 -1"/>
-    <limit lower="-1.611" upper="3.882" effort="40" velocity="6.28"/>
-  </joint>
-  <!-- Joint 2: shoulder_roll (URDF: dof_right_shoulder_roll_03) -->
-  <joint name="shoulder_roll_joint" type="revolute">
-    <parent link="shoulder_pitch_link"/>
-    <child link="shoulder_roll_link"/>
-    <origin xyz="0 -0.024250 0.080000" rpy="${pi/2} ${pi/2} 0"/>
-    <axis xyz="0 0 1"/>
-    <limit lower="-3.074" upper="0.222" effort="40" velocity="6.28"/>
-  </joint>
-  <!-- Joint 3: elbow (URDF: dof_right_shoulder_yaw_02) -->
-  <joint name="elbow_joint" type="revolute">
-    <parent link="shoulder_roll_link"/>
-    <child link="elbow_link"/>
-    <origin xyz="-0.013000 -0.142500 -0.031670" rpy="${-pi/2} 0 0"/>
-    <axis xyz="0 0 1"/>
-    <limit lower="-0.042" upper="3.096" effort="20" velocity="6.28"/>
-  </joint>
-  <!-- Joint 4: wrist_pitch (URDF: dof_right_elbow_02) -->
-  <joint name="wrist_pitch_joint" type="revolute">
-    <parent link="elbow_link"/>
-    <child link="wrist_pitch_link"/>
-    <origin xyz="0.019000 -0.010000 -0.137000" rpy="${-pi/2} 0 ${pi/2}"/>
-    <axis xyz="0 0 1"/>
-    <limit lower="-0.042" upper="0.152" effort="6" velocity="6.28"/>
-  </joint>
-  <!-- Joint 5: wrist_roll (URDF: dof_right_wrist_00) -->
-  <joint name="wrist_roll_joint" type="revolute">
-    <parent link="wrist_pitch_link"/>
-    <child link="wrist_roll_link"/>
-    <origin xyz="0.017350 0.103000 0.018000" rpy="${-pi/2} ${pi/2} 0"/>
-    <axis xyz="0 0 -1"/>
-    <limit lower="-1.887" upper="-0.002" effort="6" velocity="6.28"/>
-  </joint>
-  <!-- End-effector fixed joint -->
-  <joint name="end_effector_joint" type="fixed">
-    <parent link="wrist_roll_link"/>
-    <child link="end_effector_link"/>
-    <origin xyz="0 0 -0.05" rpy="0 0 0"/>
-  </joint>
-  <!-- ros2_control hardware tags (separate xacro) -->
+  <xacro:arg name="use_mock_hardware" default="true"/>
+  <!-- Official KBot 20-DOF model from kscalelabs/kbot-models -->
+  <xacro:include filename="$(find steveros_description)/urdf/kbot.urdf"/>
+  <!-- ros2_control hardware interface configuration -->
   <xacro:include filename="$(find steveros_description)/urdf/steveros_ros2_control.xacro"/>
 </robot>

File: steveros_description/urdf/steveros_ros2_control.xacro (robot description, xacro)
@@ -1,6 +1,5 @@
 <?xml version="1.0"?>
 <robot xmlns:xacro="http://www.ros.org/wiki/xacro">
-  <xacro:arg name="use_mock_hardware" default="true"/>
-  <ros2_control name="steveros_arm" type="system">
+  <ros2_control name="steveros_kbot" type="system">
     <hardware>
       <xacro:if value="$(arg use_mock_hardware)">
@@ -14,64 +13,243 @@
       </xacro:unless>
     </hardware>
-    <!-- Joint 1: shoulder_pitch (motor ID 21, sign +1) -->
-    <joint name="shoulder_pitch_joint">
+    <!-- ==================== RIGHT ARM ==================== -->
+    <joint name="dof_right_shoulder_pitch_03">
       <param name="motor_id">21</param>
       <param name="sign">1</param>
-      <param name="zero_offset_deg">171.22</param>
-      <command_interface name="position">
-        <param name="min">-1.611</param>
-        <param name="max">3.882</param>
-      </command_interface>
-      <state_interface name="position"/>
-      <state_interface name="velocity"/>
-      <state_interface name="effort"/>
-    </joint>
-    <!-- Joint 2: shoulder_roll (motor ID 22, sign -1) -->
-    <joint name="shoulder_roll_joint">
+      <param name="zero_offset_deg">0</param>
+      <command_interface name="position">
+        <param name="min">-3.490658</param>
+        <param name="max">1.047198</param>
+      </command_interface>
+      <state_interface name="position"/>
+      <state_interface name="velocity"/>
+      <state_interface name="effort"/>
+    </joint>
+    <joint name="dof_right_shoulder_roll_03">
       <param name="motor_id">22</param>
-      <param name="sign">-1</param>
-      <param name="zero_offset_deg">-12.69</param>
-      <command_interface name="position">
-        <param name="min">-3.074</param>
-        <param name="max">0.222</param>
-      </command_interface>
-      <state_interface name="position"/>
-      <state_interface name="velocity"/>
-      <state_interface name="effort"/>
-    </joint>
-    <!-- Joint 3: elbow (motor ID 23, sign +1) -->
-    <joint name="elbow_joint">
+      <param name="sign">1</param>
+      <param name="zero_offset_deg">0</param>
+      <command_interface name="position">
+        <param name="min">-1.658063</param>
+        <param name="max">0.436332</param>
+      </command_interface>
+      <state_interface name="position"/>
+      <state_interface name="velocity"/>
+      <state_interface name="effort"/>
+    </joint>
+    <joint name="dof_right_shoulder_yaw_02">
       <param name="motor_id">23</param>
       <param name="sign">1</param>
-      <param name="zero_offset_deg">-170.37</param>
-      <command_interface name="position">
-        <param name="min">-0.042</param>
-        <param name="max">3.096</param>
-      </command_interface>
-      <state_interface name="position"/>
-      <state_interface name="velocity"/>
-      <state_interface name="effort"/>
-    </joint>
-    <!-- Joint 4: wrist_pitch (motor ID 24, sign +1) -->
-    <joint name="wrist_pitch_joint">
+      <param name="zero_offset_deg">0</param>
+      <command_interface name="position">
+        <param name="min">-1.671886</param>
+        <param name="max">1.671886</param>
+      </command_interface>
+      <state_interface name="position"/>
+      <state_interface name="velocity"/>
+      <state_interface name="effort"/>
+    </joint>
+    <joint name="dof_right_elbow_02">
       <param name="motor_id">24</param>
       <param name="sign">1</param>
-      <param name="zero_offset_deg">280.26</param>
-      <command_interface name="position">
-        <param name="min">-0.042</param>
-        <param name="max">0.152</param>
-      </command_interface>
-      <state_interface name="position"/>
-      <state_interface name="velocity"/>
-      <state_interface name="effort"/>
-    </joint>
-    <!-- Joint 5: wrist_roll (motor ID 25, sign +1) -->
-    <joint name="wrist_roll_joint">
+      <param name="zero_offset_deg">0</param>
+      <command_interface name="position">
+        <param name="min">0</param>
+        <param name="max">2.478368</param>
+      </command_interface>
+      <state_interface name="position"/>
+      <state_interface name="velocity"/>
+      <state_interface name="effort"/>
+    </joint>
+    <joint name="dof_right_wrist_00">
       <param name="motor_id">25</param>
       <param name="sign">1</param>
-      <param name="zero_offset_deg">108.13</param>
-      <command_interface name="position">
-        <param name="min">-1.887</param>
-        <param name="max">-0.002</param>
+      <param name="zero_offset_deg">0</param>
+      <command_interface name="position">
+        <param name="min">-1.378810</param>
+        <param name="max">1.378810</param>
+      </command_interface>
+      <state_interface name="position"/>
+      <state_interface name="velocity"/>
+      <state_interface name="effort"/>
+    </joint>
+    <!-- ==================== LEFT ARM ==================== -->
+    <joint name="dof_left_shoulder_pitch_03">
+      <param name="motor_id">11</param>
+      <param name="sign">1</param>
+      <param name="zero_offset_deg">0</param>
+      <command_interface name="position">
+        <param name="min">-1.047198</param>
+        <param name="max">3.490658</param>
+      </command_interface>
+      <state_interface name="position"/>
+      <state_interface name="velocity"/>
+      <state_interface name="effort"/>
+    </joint>
+    <joint name="dof_left_shoulder_roll_03">
+      <param name="motor_id">12</param>
+      <param name="sign">1</param>
+      <param name="zero_offset_deg">0</param>
+      <command_interface name="position">
+        <param name="min">-0.436332</param>
+        <param name="max">1.658063</param>
+      </command_interface>
+      <state_interface name="position"/>
+      <state_interface name="velocity"/>
+      <state_interface name="effort"/>
+    </joint>
+    <joint name="dof_left_shoulder_yaw_02">
+      <param name="motor_id">13</param>
+      <param name="sign">1</param>
+      <param name="zero_offset_deg">0</param>
+      <command_interface name="position">
+        <param name="min">-1.671886</param>
+        <param name="max">1.671886</param>
+      </command_interface>
+      <state_interface name="position"/>
+      <state_interface name="velocity"/>
+      <state_interface name="effort"/>
+    </joint>
+    <joint name="dof_left_elbow_02">
+      <param name="motor_id">14</param>
+      <param name="sign">1</param>
+      <param name="zero_offset_deg">0</param>
+      <command_interface name="position">
+        <param name="min">-2.478368</param>
+        <param name="max">0</param>
+      </command_interface>
+      <state_interface name="position"/>
+      <state_interface name="velocity"/>
+      <state_interface name="effort"/>
+    </joint>
+    <joint name="dof_left_wrist_00">
+      <param name="motor_id">15</param>
+      <param name="sign">1</param>
+      <param name="zero_offset_deg">0</param>
+      <command_interface name="position">
+        <param name="min">-1.378810</param>
+        <param name="max">1.378810</param>
+      </command_interface>
+      <state_interface name="position"/>
+      <state_interface name="velocity"/>
+      <state_interface name="effort"/>
+    </joint>
+    <!-- ==================== RIGHT LEG ==================== -->
+    <joint name="dof_right_hip_pitch_04">
+      <param name="motor_id">41</param>
+      <param name="sign">1</param>
+      <param name="zero_offset_deg">0</param>
+      <command_interface name="position">
+        <param name="min">-2.216568</param>
+        <param name="max">1.047198</param>
+      </command_interface>
+      <state_interface name="position"/>
+      <state_interface name="velocity"/>
+      <state_interface name="effort"/>
+    </joint>
+    <joint name="dof_right_hip_roll_03">
+      <param name="motor_id">42</param>
+      <param name="sign">1</param>
+      <param name="zero_offset_deg">0</param>
+      <command_interface name="position">
+        <param name="min">-2.268928</param>
+        <param name="max">0.209440</param>
+      </command_interface>
+      <state_interface name="position"/>
+      <state_interface name="velocity"/>
+      <state_interface name="effort"/>
+    </joint>
+    <joint name="dof_right_hip_yaw_03">
+      <param name="motor_id">43</param>
+      <param name="sign">1</param>
+      <param name="zero_offset_deg">0</param>
+      <command_interface name="position">
+        <param name="min">-1.570796</param>
+        <param name="max">1.570796</param>
+      </command_interface>
+      <state_interface name="position"/>
+      <state_interface name="velocity"/>
+      <state_interface name="effort"/>
+    </joint>
+    <joint name="dof_right_knee_04">
+      <param name="motor_id">44</param>
+      <param name="sign">1</param>
+      <param name="zero_offset_deg">0</param>
+      <command_interface name="position">
+        <param name="min">-2.705260</param>
+        <param name="max">0</param>
+      </command_interface>
+      <state_interface name="position"/>
+      <state_interface name="velocity"/>
+      <state_interface name="effort"/>
+    </joint>
+    <joint name="dof_right_ankle_02">
+      <param name="motor_id">45</param>
+      <param name="sign">1</param>
+      <param name="zero_offset_deg">0</param>
+      <command_interface name="position">
+        <param name="min">-0.261799</param>
+        <param name="max">1.134464</param>
+      </command_interface>
+      <state_interface name="position"/>
+      <state_interface name="velocity"/>
+      <state_interface name="effort"/>
+    </joint>
+    <!-- ==================== LEFT LEG ==================== -->
+    <joint name="dof_left_hip_pitch_04">
+      <param name="motor_id">31</param>
+      <param name="sign">1</param>
+      <param name="zero_offset_deg">0</param>
+      <command_interface name="position">
+        <param name="min">-1.047198</param>
+        <param name="max">2.216568</param>
+      </command_interface>
+      <state_interface name="position"/>
+      <state_interface name="velocity"/>
+      <state_interface name="effort"/>
+    </joint>
+    <joint name="dof_left_hip_roll_03">
+      <param name="motor_id">32</param>
+      <param name="sign">1</param>
+      <param name="zero_offset_deg">0</param>
+      <command_interface name="position">
+        <param name="min">-0.209440</param>
+        <param name="max">2.268928</param>
+      </command_interface>
+      <state_interface name="position"/>
+      <state_interface name="velocity"/>
+      <state_interface name="effort"/>
+    </joint>
+    <joint name="dof_left_hip_yaw_03">
+      <param name="motor_id">33</param>
+      <param name="sign">1</param>
+      <param name="zero_offset_deg">0</param>
+      <command_interface name="position">
+        <param name="min">-1.570796</param>
+        <param name="max">1.570796</param>
+      </command_interface>
+      <state_interface name="position"/>
+      <state_interface name="velocity"/>
+      <state_interface name="effort"/>
+    </joint>
+    <joint name="dof_left_knee_04">
+      <param name="motor_id">34</param>
+      <param name="sign">1</param>
+      <param name="zero_offset_deg">0</param>
+      <command_interface name="position">
+        <param name="min">0</param>
+        <param name="max">2.705260</param>
+      </command_interface>
+      <state_interface name="position"/>
+      <state_interface name="velocity"/>
+      <state_interface name="effort"/>
+    </joint>
+    <joint name="dof_left_ankle_02">
+      <param name="motor_id">35</param>
+      <param name="sign">1</param>
+      <param name="zero_offset_deg">0</param>
+      <command_interface name="position">
+        <param name="min">-1.134464</param>
+        <param name="max">0.261799</param>
       </command_interface>
       <state_interface name="position"/>
