Commit message: Add MoveIt2 config and upgrade to kbot-v2 URDF with collision meshes
Replace kbot-v1 URDF/meshes with kbot-v2 from kscalelabs/kscale-assets
(adds collision geometry on all links). Create steveros_moveit_config
package with pick_ik solver (position-only for 5-DOF arms), OMPL
planners, SRDF with right_arm/left_arm planning groups, joint limits,
and launch files for both mock and real hardware.

Co-Authored-By: Claude Opus 4.6 <noreply@anthropic.com>

File: steveros_description/urdf/kbot.urdf (robot description, URDF)
Before this commit: robot assy_forurdf_kdheadless, 23 links, 22 joints
Links:
- removed link KC_C_101R_ShldYokeDrive
- removed link KC_C_401L_Up_Forearm_Drive
- removed link KD_B_102B_TORSO_BTM
- removed link KD_C_101L_ShldYokeDrive
- removed link KD_C_301L_LowerBicepDrive
- removed link KD_D_102L_L_Hip_Yoke_Drive
- removed link KD_D_102R
- removed link KD_D_301L_L_Femur_Lower_Drive
- removed link KD_D_301R
- removed link KD_D_401L_L_Shin_Drive
- removed link KD_D_401R
- removed link LFootBushing_GPF_1517_12
- removed link L_Hip_Roll_RS03
- removed link L_Hip_Roll_RS03_2
- removed link PRT0001
- removed link PRT0001_2
- removed link RFootBushing_GPF_1517_12
- removed link base
- added link KB_C_501X_Left_Bayonet_Adapter_Hard_Stop, mass 0.152198; collision mesh filename=package://steveros_description/meshes/KB_C_501X_Left_Bayone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; visual mesh filename=package://steveros_description/meshes/KB_C_501X_Left_Bayone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
- added link KB_C_501X_Right_Bayonet_Adapter_Hard_Stop, mass 0.152198; collision mesh filename=package://steveros_description/meshes/KB_C_501X_Right_Bayon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; visual mesh filename=package://steveros_description/meshes/KB_C_501X_Right_Bayon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
- added link KB_D_501L_L_LEG_FOOT, mass 0.483858; collision mesh filename=package://steveros_description/meshes/KB_D_501L_L_LEG_FOOT.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; visual mesh filename=package://steveros_description/meshes/KB_D_501L_L_LEG_FOOT.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
- added link KB_D_501R_R_LEG_FOOT, mass 0.483858; collision mesh filename=package://steveros_description/meshes/KB_D_501R_R_LEG_FOOT.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; visual mesh filename=package://steveros_description/meshes/KB_D_501R_R_LEG_FOOT.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
- added link KC_C_104L_PitchHardstopDriven, mass 0.584843; collision mesh filename=package://steveros_description/meshes/KC_C_104L_PitchHardst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; visual mesh filename=package://steveros_description/meshes/KC_C_104L_PitchHardst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
- added link KC_C_104R_PitchHardstopDriven, mass 0.584848; collision mesh filename=package://steveros_description/meshes/KC_C_104R_PitchHardst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; visual mesh filename=package://steveros_description/meshes/KC_C_104R_PitchHardst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
- added link KC_C_202L, mass 0.579259; collision mesh filename=package://steveros_description/meshes/KC_C_202L.collision.s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; visual mesh filename=package://steveros_description/meshes/KC_C_202L.stl
- added link KC_C_401L_L_UpForearmDrive, mass 0.585219; collision mesh filename=package://steveros_description/meshes/KC_C_401L_L_UpForearm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; visual mesh filename=package://steveros_description/meshes/KC_C_401L_L_UpForearm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
- added link KC_D_102L_L_Hip_Yoke_Drive, mass 0.530424; collision mesh filename=package://steveros_description/meshes/KC_D_102L_L_Hip_Yoke_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; visual mesh filename=package://steveros_description/meshes/KC_D_102L_L_Hip_Yoke_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
- added link KC_D_102R_R_Hip_Yoke_Drive, mass 0.530428; collision mesh filename=package://steveros_description/meshes/KC_D_102R_R_Hip_Yoke_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; visual mesh filename=package://steveros_description/meshes/KC_D_102R_R_Hip_Yoke_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
- added link KC_D_301L_L_Femur_Lower_Drive, mass 2.343629; collision mesh filename=package://steveros_description/meshes/KC_D_301L_L_Femur_Low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; visual mesh filename=package://steveros_description/meshes/KC_D_301L_L_Femur_Low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
- added link KC_D_301R_R_Femur_Lower_Drive, mass 2.343635; collision mesh filename=package://steveros_description/meshes/KC_D_301R_R_Femur_Low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; visual mesh filename=package://steveros_description/meshes/KC_D_301R_R_Femur_Low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
- added link KC_D_401L_L_Shin_Drive, mass 1.670535; collision mesh filename=package://steveros_description/meshes/KC_D_401L_L_Shin_Driv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; visual mesh filename=package://steveros_description/meshes/KC_D_401L_L_Shin_Driv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
- added link KC_D_401R_R_Shin_Drive, mass 1.670592; collision mesh filename=package://steveros_description/meshes/KC_D_401R_R_Shin_Driv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; visual mesh filename=package://steveros_description/meshes/KC_D_401R_R_Shin_Driv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
- added link RS03_5, mass 2.373239; collision mesh filename=package://steveros_description/meshes/RS03_5.collision.stl; visual mesh filename=package://steveros_description/meshes/RS03_5.stl
- added link RS03_6, mass 1.676479; collision mesh filename=package://steveros_description/meshes/RS03_6.collision.stl; visual mesh filename=package://steveros_description/meshes/RS03_6.stl
- added link Torso_Side_Right, mass 13.516427; collision mesh filename=package://steveros_description/meshes/Torso_Side_Right.coll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; visual mesh filename=package://steveros_description/meshes/Torso_Side_Right.stl
- added link floating_base_link, mass 0.001; visual sphere radius=0.01
- link KC_C_202R: mass 0.753224 -> 0.743508; geometry collision mesh filename=package://steveros_description/meshes/KC_C_202R.collision.s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; visual mesh filename=package://steveros_description/meshes/KC_C_202R.stl
- link KC_C_401R_R_UpForearmDrive: mass 0.641859 -> 0.585204; geometry collision mesh filename=package://steveros_description/meshes/KC_C_401R_R_UpForearm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; visual mesh filename=package://steveros_description/meshes/KC_C_401R_R_UpForearm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
- link RS03_3: mass 1.789232 -> 1.676509; geometry collision mesh filename=package://steveros_description/meshes/RS03_3.collision.stl; visual mesh filename=package://steveros_description/meshes/RS03_3.stl
- link RS03_4: mass 1.789190 -> 2.373184; geometry collision mesh filename=package://steveros_description/meshes/RS03_4.collision.stl; visual mesh filename=package://steveros_description/meshes/RS03_4.stl
- link imu: geometry collision mesh filename=package://steveros_description/meshes/imu.collision.stl; visual mesh filename=package://steveros_description/meshes/imu.stl
Joints:
- removed joint base_joint
- added joint floating_base_joint: type fixed, parent floating_base_link, child Torso_Side_Right, origin xyz=0 0 0 rpy=0.00 0.00 1.57
- joint dof_left_ankle_02: child LFootBushing_GPF_1517_12 -> KB_D_501L_L_LEG_FOOT; limit lower=-1.134464 upper=0.261799 effort=17 velocity=37.699 -> lower=-1.256637 upper=0.226893 effort=17 velocity=37.699; origin xyz=-0.030000 -0.290000 0.000950 rpy=3.141593 0 0 -> xyz=-0.030000 -0.290000 0.035100 rpy=-3.141593 0 0; parent KD_D_401L_L_Shin_Drive -> KC_D_401L_L_Shin_Drive
- joint dof_left_elbow_02: axis 0 0 1 -> 0 0 -1; child KC_C_401L_Up_Forearm_Drive -> KC_C_401L_L_UpForearmDrive; origin xyz=-0.019000 -0.010000 -0.137000 rpy=1.570796 0 1.570796 -> xyz=-0.018500 0.010000 0.137000 rpy=-3.141593 1.570796 0; parent KD_C_301L_LowerBicepDrive -> KC_C_202L
- joint dof_left_hip_pitch_04: child KD_D_102L_L_Hip_Yoke_Drive -> KC_D_102L_L_Hip_Yoke_Drive; origin xyz=0.056001 0.002025 -0.073841 rpy=-1.570796 0 1.570796 -> xyz=0.147969 0.000007 -0.284479 rpy=-1.570796 0 1.570796; parent KD_B_102B_TORSO_BTM -> Torso_Side_Right
- joint dof_left_hip_roll_03: child L_Hip_Roll_RS03 -> RS03_5; origin xyz=-0.028250 0.030000 -0.071000 rpy=3.141593 -1.570796 0 -> xyz=-0.028250 0.030000 -0.071000 rpy=0 1.570796 0; parent KD_D_102L_L_Hip_Yoke_Drive -> KC_D_102L_L_Hip_Yoke_Drive
- joint dof_left_hip_yaw_03: axis 0 0 1 -> 0 0 -1; child KD_D_301L_L_Femur_Lower_Drive -> KC_D_301L_L_Femur_Lower_Drive; origin xyz=0 -0.143000 0.025250 rpy=1.570796 0 -3.141593 -> xyz=0 0.143000 0.024250 rpy=-1.570796 0 0; parent L_Hip_Roll_RS03 -> RS03_5
- joint dof_left_knee_04: child KD_D_401L_L_Shin_Drive -> KC_D_401L_L_Shin_Drive; origin xyz=-0.021000 0.021000 -0.212000 rpy=1.570796 0 1.570796 -> xyz=-0.020500 -0.021000 0.212000 rpy=-1.570796 0 -1.570796; parent KD_D_301L_L_Femur_Lower_Drive -> KC_D_301L_L_Femur_Lower_Drive
- joint dof_left_shoulder_pitch_03: axis 0 0 -1 -> 0 0 1; child KD_C_101L_ShldYokeDrive -> KC_C_104L_PitchHardstopDriven; origin xyz=0.121001 0.002025 0.336659 rpy=0 1.570796 0 -> xyz=0.213969 0.000007 0.126021 rpy=-1.570796 0 1.570796; parent KD_B_102B_TORSO_BTM -> Torso_Side_Right
- joint dof_left_shoulder_roll_03: child RS03_4 -> RS03_6; limit lower=-0.436332 upper=1.658063 effort=60 velocity=18.849 -> lower=-0.383972 upper=1.658063 effort=60 velocity=18.849; origin xyz=0 -0.024250 0.080000 rpy=1.570796 -1.570796 0 -> xyz=-0.024250 0 -0.080000 rpy=-3.141593 1.570796 0; parent KD_C_101L_ShldYokeDrive -> KC_C_104L_PitchHardstopDriven
- joint dof_left_shoulder_yaw_02: axis 0 0 1 -> 0 0 -1; child KD_C_301L_LowerBicepDrive -> KC_C_202L; limit lower=-1.671886 upper=1.671886 effort=17 velocity=37.699 -> lower=-1.658063 upper=1.658063 effort=17 velocity=37.699; origin xyz=0.013000 -0.142500 -0.030750 rpy=-1.570796 0 0 -> xyz=0.013000 -0.142000 -0.030250 rpy=1.570796 0 0; parent RS03_4 -> RS03_6
- joint dof_left_wrist_00: child PRT0001_2 -> KB_C_501X_Left_Bayonet_Adapter_Hard_Stop; limit lower=-1.378810 upper=1.378810 effort=14 velocity=27.227 -> lower=-1.745329 upper=1.745329 effort=14 velocity=27.227; origin xyz=0.017350 -0.103000 0.018000 rpy=1.570796 -1.570796 0 -> xyz=-0.103000 0.017350 -0.018000 rpy=-3.141593 1.570796 0; parent KC_C_401L_Up_Forearm_Drive -> KC_C_401L_L_UpForearmDrive
- joint dof_right_ankle_02: axis 0 0 -1 -> 0 0 1; child RFootBushing_GPF_1517_12 -> KB_D_501R_R_LEG_FOOT; limit lower=-0.261799 upper=1.134464 effort=17 velocity=37.699 -> lower=-0.226893 upper=1.256637 effort=17 velocity=37.699; origin xyz=-0.030000 -0.290000 -0.000950 rpy=0 0 0 -> xyz=-0.030000 0.290000 0.035100 rpy=0 0 0; parent KD_D_401R -> KC_D_401R_R_Shin_Drive
- joint dof_right_elbow_02: axis 0 0 1 -> 0 0 -1; origin xyz=0.019000 -0.010000 -0.137000 rpy=-1.570796 0 1.570796 -> xyz=0.018500 -0.010000 -0.137000 rpy=0 1.570796 0
- joint dof_right_hip_pitch_04: child KD_D_102R -> KC_D_102R_R_Hip_Yoke_Drive; origin xyz=-0.055999 0.002025 -0.073841 rpy=1.570796 0 1.570796 -> xyz=0.037469 0.000007 -0.284479 rpy=1.570796 0 1.570796; parent KD_B_102B_TORSO_BTM -> Torso_Side_Right
- joint dof_right_hip_roll_03: axis 0 0 1 -> 0 0 -1; child L_Hip_Roll_RS03_2 -> RS03_4; origin xyz=-0.028250 -0.030000 -0.071000 rpy=0 -1.570796 0 -> xyz=-0.028250 -0.030000 -0.071000 rpy=3.141593 -1.570796 0; parent KD_D_102R -> KC_D_102R_R_Hip_Yoke_Drive
- joint dof_right_hip_yaw_03: axis 0 0 1 -> 0 0 -1; child KD_D_301R -> KC_D_301R_R_Femur_Lower_Drive; origin xyz=0 -0.143000 -0.025250 rpy=-1.570796 0 0 -> xyz=0 0.143000 0.024250 rpy=-1.570796 0 0; parent L_Hip_Roll_RS03_2 -> RS03_4
- joint dof_right_knee_04: axis 0 0 -1 -> 0 0 1; child KD_D_401R -> KC_D_401R_R_Shin_Drive; origin xyz=0.021000 0.021000 -0.212000 rpy=1.570796 0 1.570796 -> xyz=0.020500 -0.021000 0.212000 rpy=1.570796 0 -1.570796; parent KD_D_301R -> KC_D_301R_R_Femur_Lower_Drive
- joint dof_right_shoulder_pitch_03: axis 0 0 -1 -> 0 0 1; child KC_C_101R_ShldYokeDrive -> KC_C_104R_PitchHardstopDriven; limit lower=-3.490658 upper=1.047198 effort=60 velocity=18.849 -> lower=-2.617994 upper=2.094395 effort=60 velocity=18.849; origin xyz=-0.120999 0.002025 0.336659 rpy=0 -1.570796 0 -> xyz=-0.028031 0.000007 0.126021 rpy=1.570796 0 1.570796; parent KD_B_102B_TORSO_BTM -> Torso_Side_Right
- joint dof_right_shoulder_roll_03: axis 0 0 1 -> 0 0 -1; limit lower=-1.658063 upper=0.436332 effort=60 velocity=18.849 -> lower=-1.658063 upper=0.383972 effort=60 velocity=18.849; origin xyz=0 -0.024250 0.080000 rpy=1.570796 1.570796 0 -> xyz=-0.024250 0 -0.080000 rpy=-3.141593 -1.570796 0; parent KC_C_101R_ShldYokeDrive -> KC_C_104R_PitchHardstopDriven
- joint dof_right_shoulder_yaw_02: limit lower=-1.671886 upper=1.671886 effort=17 velocity=37.699 -> lower=-1.658063 upper=1.658063 effort=17 velocity=37.699; origin xyz=-0.013000 -0.142500 -0.031670 rpy=-1.570796 0 0 -> xyz=-0.013000 0.142000 0.030250 rpy=1.570796 0 0
- joint dof_right_wrist_00: axis 0 0 -1 -> 0 0 1; child PRT0001 -> KB_C_501X_Right_Bayonet_Adapter_Hard_Stop; limit lower=-1.378810 upper=1.378810 effort=14 velocity=27.227 -> lower=-1.745329 upper=1.745329 effort=14 velocity=27.227; origin xyz=0.017350 0.103000 0.018000 rpy=-1.570796 1.570796 0 -> xyz=0.103000 0.017350 -0.018000 rpy=0 -1.570796 0
- joint frame_imu_site: origin xyz=0.003707 -0.010539 0.394701 rpy=0.011111 0 0 -> xyz=0.121783 0.043292 0.231518 rpy=1.582557 1.570794 1.582557; parent KD_B_102B_TORSO_BTM -> Torso_Side_Right
