Commit message: Update robot model to KD-series URDF with tuned PD gains
New URDF export (assy_forurdf_kdheadless) with updated link/mesh names,
joint origins, axes, and limits. Tuned PD gains from kbot-v2 metadata.
Updated SRDF collision config and meshes to match.

Source: https://github.com/kscalelabs/kbot-models/tree/master/kbot-full-collisions

Co-Authored-By: Claude Opus 4.6 <noreply@anthropic.com>

File: steveros_description/urdf/kbot.urdf (robot description, URDF)
Before this commit: robot kbotv2p0_nohands, 23 links, 22 joints
Links:
- removed link KB_C_501X_Left_Bayonet_Adapter_Hard_Stop
- removed link KB_C_501X_Right_Bayonet_Adapter_Hard_Stop
- removed link KB_D_501L_L_LEG_FOOT
- removed link KB_D_501R_R_LEG_FOOT
- removed link KC_C_104L_PitchHardstopDriven
- removed link KC_C_104R_PitchHardstopDriven
- removed link KC_C_202L
- removed link KC_C_401L_L_UpForearmDrive
- removed link KC_D_102L_L_Hip_Yoke_Drive
- removed link KC_D_102R_R_Hip_Yoke_Drive
- removed link KC_D_301L_L_Femur_Lower_Drive
- removed link KC_D_301R_R_Femur_Lower_Drive
- removed link KC_D_401L_L_Shin_Drive
- removed link KC_D_401R_R_Shin_Drive
- removed link RS03_5
- removed link RS03_6
- removed link Torso_Side_Right
- removed link floating_base_link
- added link KC_C_101R_ShldYokeDrive, mass 0.569870; collision mesh filename=package://steveros_description/meshes/KC_C_101R_ShldYokeDri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; visual mesh filename=package://steveros_description/meshes/KC_C_101R_ShldYokeDri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
- added link KC_C_401L_Up_Forearm_Drive, mass 0.641873; collision mesh filename=package://steveros_description/meshes/KC_C_401L_Up_Forearm_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; visual mesh filename=package://steveros_description/meshes/KC_C_401L_Up_Forearm_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
- added link KD_B_102B_TORSO_BTM, mass 12.968840; collision mesh filename=package://steveros_description/meshes/KD_B_102B_TORSO_BTM.c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; visual mesh filename=package://steveros_description/meshes/KD_B_102B_TORSO_BTM.s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
- added link KD_C_101L_ShldYokeDrive, mass 0.569863; collision mesh filename=package://steveros_description/meshes/KD_C_101L_ShldYokeDri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; visual mesh filename=package://steveros_description/meshes/KD_C_101L_ShldYokeDri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
- added link KD_C_301L_LowerBicepDrive, mass 0.866827; collision mesh filename=package://steveros_description/meshes/KD_C_301L_LowerBicepD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; visual mesh filename=package://steveros_description/meshes/KD_C_301L_LowerBicepD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
- added link KD_D_102L_L_Hip_Yoke_Drive, mass 0.550354; collision mesh filename=package://steveros_description/meshes/KD_D_102L_L_Hip_Yoke_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; visual mesh filename=package://steveros_description/meshes/KD_D_102L_L_Hip_Yoke_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
- added link KD_D_102R, mass 0.550361; collision mesh filename=package://steveros_description/meshes/KD_D_102R.collision.s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; visual mesh filename=package://steveros_description/meshes/KD_D_102R.stl
- added link KD_D_301L_L_Femur_Lower_Drive, mass 2.349254; collision mesh filename=package://steveros_description/meshes/KD_D_301L_L_Femur_Low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; visual mesh filename=package://steveros_description/meshes/KD_D_301L_L_Femur_Low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
- added link KD_D_301R, mass 2.349261; collision mesh filename=package://steveros_description/meshes/KD_D_301R.collision.s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; visual mesh filename=package://steveros_description/meshes/KD_D_301R.stl
- added link KD_D_401L_L_Shin_Drive, mass 1.684707; collision mesh filename=package://steveros_description/meshes/KD_D_401L_L_Shin_Driv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; visual mesh filename=package://steveros_description/meshes/KD_D_401L_L_Shin_Driv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
- added link KD_D_401R, mass 1.684717; collision mesh filename=package://steveros_description/meshes/KD_D_401R.collision.s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; visual mesh filename=package://steveros_description/meshes/KD_D_401R.stl
- added link LFootBushing_GPF_1517_12, mass 0.608966; collision mesh filename=package://steveros_description/meshes/LFootBushing_GPF_1517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; visual mesh filename=package://steveros_description/meshes/LFootBushing_GPF_1517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
- added link L_Hip_Roll_RS03, mass 2.396969; collision mesh filename=package://steveros_description/meshes/L_Hip_Roll_RS03.colli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; visual mesh filename=package://steveros_description/meshes/L_Hip_Roll_RS03.stl
- added link L_Hip_Roll_RS03_2, mass 2.396917; collision mesh filename=package://steveros_description/meshes/L_Hip_Roll_RS03_2.col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; visual mesh filename=package://steveros_description/meshes/L_Hip_Roll_RS03_2.stl
- added link PRT0001, mass 0.469028; collision mesh filename=package://steveros_description/meshes/PRT0001.collision.stl; visual mesh filename=package://steveros_description/meshes/PRT0001.stl
- added link PRT0001_2, mass 0.469028; collision mesh filename=package://steveros_description/meshes/PRT0001_2.collision.s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; visual mesh filename=package://steveros_description/meshes/PRT0001_2.stl
- added link RFootBushing_GPF_1517_12, mass 0.608742; collision mesh filename=package://steveros_description/meshes/RFootBushing_GPF_1517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; visual mesh filename=package://steveros_description/meshes/RFootBushing_GPF_1517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
- added link base, mass 0.001; visual sphere radius=0.01
- link KC_C_202R: mass 0.743508 -> 0.753224
- link KC_C_401R_R_UpForearmDrive: mass 0.585204 -> 0.641859
- link RS03_3: mass 1.676509 -> 1.789232
- link RS03_4: mass 2.373184 -> 1.789190
Joints:
- removed joint floating_base_joint
- added joint base_joint: type fixed, parent base, child KD_B_102B_TORSO_BTM, origin xyz=0 0 0 rpy=0 0 1.5708
- joint dof_left_ankle_02: child KB_D_501L_L_LEG_FOOT -> LFootBushing_GPF_1517_12; limit lower=-1.256637 upper=0.226893 effort=17 velocity=37.699 -> lower=-1.134464 upper=0.261799 effort=17 velocity=37.699; origin xyz=-0.030000 -0.290000 0.035100 rpy=-3.141593 0 0 -> xyz=-0.030000 -0.290000 0.000950 rpy=3.141593 0 0; parent KC_D_401L_L_Shin_Drive -> KD_D_401L_L_Shin_Drive
- joint dof_left_elbow_02: axis 0 0 -1 -> 0 0 1; child KC_C_401L_L_UpForearmDrive -> KC_C_401L_Up_Forearm_Drive; origin xyz=-0.018500 0.010000 0.137000 rpy=-3.141593 1.570796 0 -> xyz=-0.019000 -0.010000 -0.137000 rpy=1.570796 0 1.570796; parent KC_C_202L -> KD_C_301L_LowerBicepDrive
- joint dof_left_hip_pitch_04: child KC_D_102L_L_Hip_Yoke_Drive -> KD_D_102L_L_Hip_Yoke_Drive; origin xyz=0.147969 0.000007 -0.284479 rpy=-1.570796 0 1.570796 -> xyz=0.056001 0.002025 -0.073841 rpy=-1.570796 0 1.570796; parent Torso_Side_Right -> KD_B_102B_TORSO_BTM
- joint dof_left_hip_roll_03: child RS03_5 -> L_Hip_Roll_RS03; origin xyz=-0.028250 0.030000 -0.071000 rpy=0 1.570796 0 -> xyz=-0.028250 0.030000 -0.071000 rpy=3.141593 -1.570796 0; parent KC_D_102L_L_Hip_Yoke_Drive -> KD_D_102L_L_Hip_Yoke_Drive
- joint dof_left_hip_yaw_03: axis 0 0 -1 -> 0 0 1; child KC_D_301L_L_Femur_Lower_Drive -> KD_D_301L_L_Femur_Lower_Drive; origin xyz=0 0.143000 0.024250 rpy=-1.570796 0 0 -> xyz=0 -0.143000 0.025250 rpy=1.570796 0 -3.141593; parent RS03_5 -> L_Hip_Roll_RS03
- joint dof_left_knee_04: child KC_D_401L_L_Shin_Drive -> KD_D_401L_L_Shin_Drive; origin xyz=-0.020500 -0.021000 0.212000 rpy=-1.570796 0 -1.570796 -> xyz=-0.021000 0.021000 -0.212000 rpy=1.570796 0 1.570796; parent KC_D_301L_L_Femur_Lower_Drive -> KD_D_301L_L_Femur_Lower_Drive
- joint dof_left_shoulder_pitch_03: axis 0 0 1 -> 0 0 -1; child KC_C_104L_PitchHardstopDriven -> KD_C_101L_ShldYokeDrive; origin xyz=0.213969 0.000007 0.126021 rpy=-1.570796 0 1.570796 -> xyz=0.121001 0.002025 0.336659 rpy=0 1.570796 0; parent Torso_Side_Right -> KD_B_102B_TORSO_BTM
- joint dof_left_shoulder_roll_03: child RS03_6 -> RS03_4; limit lower=-0.383972 upper=1.658063 effort=60 velocity=18.849 -> lower=-0.436332 upper=1.658063 effort=60 velocity=18.849; origin xyz=-0.024250 0 -0.080000 rpy=-3.141593 1.570796 0 -> xyz=0 -0.024250 0.080000 rpy=1.570796 -1.570796 0; parent KC_C_104L_PitchHardstopDriven -> KD_C_101L_ShldYokeDrive
- joint dof_left_shoulder_yaw_02: axis 0 0 -1 -> 0 0 1; child KC_C_202L -> KD_C_301L_LowerBicepDrive; limit lower=-1.658063 upper=1.658063 effort=17 velocity=37.699 -> lower=-1.671886 upper=1.671886 effort=17 velocity=37.699; origin xyz=0.013000 -0.142000 -0.030250 rpy=1.570796 0 0 -> xyz=0.013000 -0.142500 -0.030750 rpy=-1.570796 0 0; parent RS03_6 -> RS03_4
- joint dof_left_wrist_00: child KB_C_501X_Left_Bayonet_Adapter_Hard_Stop -> PRT0001_2; limit lower=-1.745329 upper=1.745329 effort=14 velocity=27.227 -> lower=-1.378810 upper=1.378810 effort=14 velocity=27.227; origin xyz=-0.103000 0.017350 -0.018000 rpy=-3.141593 1.570796 0 -> xyz=0.017350 -0.103000 0.018000 rpy=1.570796 -1.570796 0; parent KC_C_401L_L_UpForearmDrive -> KC_C_401L_Up_Forearm_Drive
- joint dof_right_ankle_02: axis 0 0 1 -> 0 0 -1; child KB_D_501R_R_LEG_FOOT -> RFootBushing_GPF_1517_12; limit lower=-0.226893 upper=1.256637 effort=17 velocity=37.699 -> lower=-0.261799 upper=1.134464 effort=17 velocity=37.699; origin xyz=-0.030000 0.290000 0.035100 rpy=0 0 0 -> xyz=-0.030000 -0.290000 -0.000950 rpy=0 0 0; parent KC_D_401R_R_Shin_Drive -> KD_D_401R
- joint dof_right_elbow_02: axis 0 0 -1 -> 0 0 1; origin xyz=0.018500 -0.010000 -0.137000 rpy=0 1.570796 0 -> xyz=0.019000 -0.010000 -0.137000 rpy=-1.570796 0 1.570796
- joint dof_right_hip_pitch_04: child KC_D_102R_R_Hip_Yoke_Drive -> KD_D_102R; origin xyz=0.037469 0.000007 -0.284479 rpy=1.570796 0 1.570796 -> xyz=-0.055999 0.002025 -0.073841 rpy=1.570796 0 1.570796; parent Torso_Side_Right -> KD_B_102B_TORSO_BTM
- joint dof_right_hip_roll_03: axis 0 0 -1 -> 0 0 1; child RS03_4 -> L_Hip_Roll_RS03_2; origin xyz=-0.028250 -0.030000 -0.071000 rpy=3.141593 -1.570796 0 -> xyz=-0.028250 -0.030000 -0.071000 rpy=0 -1.570796 0; parent KC_D_102R_R_Hip_Yoke_Drive -> KD_D_102R
- joint dof_right_hip_yaw_03: axis 0 0 -1 -> 0 0 1; child KC_D_301R_R_Femur_Lower_Drive -> KD_D_301R; origin xyz=0 0.143000 0.024250 rpy=-1.570796 0 0 -> xyz=0 -0.143000 -0.025250 rpy=-1.570796 0 0; parent RS03_4 -> L_Hip_Roll_RS03_2
- joint dof_right_knee_04: axis 0 0 1 -> 0 0 -1; child KC_D_401R_R_Shin_Drive -> KD_D_401R; origin xyz=0.020500 -0.021000 0.212000 rpy=1.570796 0 -1.570796 -> xyz=0.021000 0.021000 -0.212000 rpy=1.570796 0 1.570796; parent KC_D_301R_R_Femur_Lower_Drive -> KD_D_301R
- joint dof_right_shoulder_pitch_03: axis 0 0 1 -> 0 0 -1; child KC_C_104R_PitchHardstopDriven -> KC_C_101R_ShldYokeDrive; limit lower=-2.617994 upper=2.094395 effort=60 velocity=18.849 -> lower=-3.490658 upper=1.047198 effort=60 velocity=18.849; origin xyz=-0.028031 0.000007 0.126021 rpy=1.570796 0 1.570796 -> xyz=-0.120999 0.002025 0.336659 rpy=0 -1.570796 0; parent Torso_Side_Right -> KD_B_102B_TORSO_BTM
- joint dof_right_shoulder_roll_03: axis 0 0 -1 -> 0 0 1; limit lower=-1.658063 upper=0.383972 effort=60 velocity=18.849 -> lower=-1.658063 upper=0.436332 effort=60 velocity=18.849; origin xyz=-0.024250 0 -0.080000 rpy=-3.141593 -1.570796 0 -> xyz=0 -0.024250 0.080000 rpy=1.570796 1.570796 0; parent KC_C_104R_PitchHardstopDriven -> KC_C_101R_ShldYokeDrive
- joint dof_right_shoulder_yaw_02: limit lower=-1.658063 upper=1.658063 effort=17 velocity=37.699 -> lower=-1.671886 upper=1.671886 effort=17 velocity=37.699; origin xyz=-0.013000 0.142000 0.030250 rpy=1.570796 0 0 -> xyz=-0.013000 -0.142500 -0.031670 rpy=-1.570796 0 0
- joint dof_right_wrist_00: axis 0 0 1 -> 0 0 -1; child KB_C_501X_Right_Bayonet_Adapter_Hard_Stop -> PRT0001; limit lower=-1.745329 upper=1.745329 effort=14 velocity=27.227 -> lower=-1.378810 upper=1.378810 effort=14 velocity=27.227; origin xyz=0.103000 0.017350 -0.018000 rpy=0 -1.570796 0 -> xyz=0.017350 0.103000 0.018000 rpy=-1.570796 1.570796 0
- joint frame_imu_site: origin xyz=0.121783 0.043292 0.231518 rpy=1.582557 1.570794 1.582557 -> xyz=0.003707 -0.010539 0.394701 rpy=0.011111 0 0; parent Torso_Side_Right -> KD_B_102B_TORSO_BTM

File: steveros_description/urdf/steveros_ros2_control.xacro (robot description, xacro)
@@ -26,6 +26,6 @@
       <param name="sign">1</param>
       <param name="zero_offset_deg">112.30</param>
-      <param name="kp">40.0</param>
-      <param name="kd">4.0</param>
+      <param name="kp">100.0</param>
+      <param name="kd">8.284</param>
       <command_interface name="position">
         <param name="min">-3.490658</param>
@@ -42,6 +42,6 @@
       <param name="sign">1</param>
       <param name="zero_offset_deg">76.50</param>
-      <param name="kp">40.0</param>
-      <param name="kd">4.0</param>
+      <param name="kp">100.0</param>
+      <param name="kd">8.257</param>
       <command_interface name="position">
         <param name="min">-1.658063</param>
@@ -58,6 +58,6 @@
       <param name="sign">1</param>
       <param name="zero_offset_deg">283.93</param>
-      <param name="kp">30.0</param>
-      <param name="kd">1.0</param>
+      <param name="kp">40.0</param>
+      <param name="kd">0.945</param>
       <command_interface name="position">
         <param name="min">-1.671886</param>
@@ -74,6 +74,6 @@
       <param name="sign">1</param>
       <param name="zero_offset_deg">280.25</param>
-      <param name="kp">30.0</param>
-      <param name="kd">1.0</param>
+      <param name="kp">40.0</param>
+      <param name="kd">1.266</param>
       <command_interface name="position">
         <param name="min">0</param>
@@ -91,5 +91,5 @@
       <param name="zero_offset_deg">144.07</param>
       <param name="kp">20.0</param>
-      <param name="kd">0.5</param>
+      <param name="kd">0.295</param>
       <command_interface name="position">
         <param name="min">-1.378810</param>
@@ -107,6 +107,6 @@
       <param name="sign">1</param>
       <param name="zero_offset_deg">235.88</param>
-      <param name="kp">40.0</param>
-      <param name="kd">4.0</param>
+      <param name="kp">100.0</param>
+      <param name="kd">8.284</param>
       <command_interface name="position">
         <param name="min">-1.047198</param>
@@ -123,6 +123,6 @@
       <param name="sign">1</param>
       <param name="zero_offset_deg">83.68</param>
-      <param name="kp">40.0</param>
-      <param name="kd">4.0</param>
+      <param name="kp">100.0</param>
+      <param name="kd">8.257</param>
       <command_interface name="position">
         <param name="min">-0.436332</param>
@@ -139,6 +139,6 @@
       <param name="sign">1</param>
       <param name="zero_offset_deg">194.88</param>
-      <param name="kp">30.0</param>
-      <param name="kd">1.0</param>
+      <param name="kp">40.0</param>
+      <param name="kd">0.945</param>
       <command_interface name="position">
         <param name="min">-1.671886</param>
@@ -155,6 +155,6 @@
       <param name="sign">1</param>
       <param name="zero_offset_deg">169.29</param>
-      <param name="kp">30.0</param>
-      <param name="kd">1.0</param>
+      <param name="kp">40.0</param>
+      <param name="kd">1.266</param>
       <command_interface name="position">
         <param name="min">-2.478368</param>
@@ -172,5 +172,5 @@
       <param name="zero_offset_deg">4.01</param>
       <param name="kp">20.0</param>
-      <param name="kd">0.5</param>
+      <param name="kd">0.295</param>
       <command_interface name="position">
         <param name="min">-1.378810</param>
@@ -188,6 +188,6 @@
       <param name="sign">1</param>
       <param name="zero_offset_deg">0</param>
-      <param name="kp">85.0</param>
-      <param name="kd">5.0</param>
+      <param name="kp">150.0</param>
+      <param name="kd">24.722</param>
       <command_interface name="position">
         <param name="min">-2.216568</param>
@@ -204,6 +204,6 @@
       <param name="sign">1</param>
       <param name="zero_offset_deg">0</param>
-      <param name="kp">40.0</param>
-      <param name="kd">4.0</param>
+      <param name="kp">200.0</param>
+      <param name="kd">26.387</param>
       <command_interface name="position">
         <param name="min">-2.268928</param>
@@ -220,6 +220,6 @@
       <param name="sign">1</param>
       <param name="zero_offset_deg">0</param>
-      <param name="kp">40.0</param>
-      <param name="kd">4.0</param>
+      <param name="kp">100.0</param>
+      <param name="kd">3.419</param>
       <command_interface name="position">
         <param name="min">-1.570796</param>
@@ -236,6 +236,6 @@
       <param name="sign">1</param>
       <param name="zero_offset_deg">0</param>
-      <param name="kp">85.0</param>
-      <param name="kd">5.0</param>
+      <param name="kp">150.0</param>
+      <param name="kd">8.654</param>
       <command_interface name="position">
         <param name="min">-2.705260</param>
@@ -252,6 +252,6 @@
       <param name="sign">1</param>
       <param name="zero_offset_deg">0</param>
-      <param name="kp">30.0</param>
-      <param name="kd">1.0</param>
+      <param name="kp">40.0</param>
+      <param name="kd">0.990</param>
       <command_interface name="position">
         <param name="min">-0.261799</param>
@@ -269,6 +269,6 @@
       <param name="sign">1</param>
       <param name="zero_offset_deg">0</param>
-      <param name="kp">85.0</param>
-      <param name="kd">5.0</param>
+      <param name="kp">150.0</param>
+      <param name="kd">24.722</param>
       <command_interface name="position">
         <param name="min">-1.047198</param>
@@ -285,6 +285,6 @@
       <param name="sign">1</param>
       <param name="zero_offset_deg">0</param>
-      <param name="kp">40.0</param>
-      <param name="kd">4.0</param>
+      <param name="kp">200.0</param>
+      <param name="kd">26.387</param>
       <command_interface name="position">
         <param name="min">-0.209440</param>
@@ -301,6 +301,6 @@
       <param name="sign">1</param>
       <param name="zero_offset_deg">0</param>
-      <param name="kp">40.0</param>
-      <param name="kd">4.0</param>
+      <param name="kp">100.0</param>
+      <param name="kd">3.419</param>
       <command_interface name="position">
         <param name="min">-1.570796</param>
@@ -317,6 +317,6 @@
       <param name="sign">1</param>
       <param name="zero_offset_deg">0</param>
-      <param name="kp">85.0</param>
-      <param name="kd">5.0</param>
+      <param name="kp">150.0</param>
+      <param name="kd">8.654</param>
       <command_interface name="position">
         <param name="min">0</param>
@@ -333,6 +333,6 @@
       <param name="sign">1</param>
       <param name="zero_offset_deg">0</param>
-      <param name="kp">30.0</param>
-      <param name="kd">1.0</param>
+      <param name="kp">40.0</param>
+      <param name="kd">0.990</param>
       <command_interface name="position">
         <param name="min">-1.134464</param>
